File: ELECTRONICS/coreBoard/coreBoard.kicad_sch (KiCad schematic)
At the start: 0 parts

Commit message: Konnect test
Parts:
- added Bt_Guide1, Bt_L_A1, Bt_L_D1, Bt_L_LB1, Bt_L_S1, Bt_L_W1, Bt_Menu1, Bt_R_A1, Bt_R_B1, Bt_R_RB1, Bt_R_X1, Bt_R_Y1, Bt_Share1, Bt_View1: 1825910-6, Tactile Switch - TE 1825910_6:SW4_1825910-B_TEC, symbol Tactile Switch - TE 1825910_6:1825910-6
- added C1, C2, C3, C4, C5, C6, C7, C8: 100nF, Capacitor_THT:C_Disc_D5.0mm_W2.5mm_P5.00mm, symbol Device:C
- added LED1, LED2, LED3, LED4, LED5, LED6, LED7, LED8: WS2812B, LED_THT:LED_D5.0mm-4_RGB, symbol LED:WS2812B
- added R1, R10, R11, R12, R13, R14, R15, R16, R2, R3, R4, R5, R6, R7, R8, R9: 10k, Resistor_THT:R_Axial_DIN0207_L6.3mm_D2.5mm_P10.16mm_Horizontal, symbol Device:R
- added R17: 470, Resistor_THT:R_Axial_DIN0207_L6.3mm_D2.5mm_P10.16mm_Horizontal, symbol Device:R
- added RP1: RaspberryPi_Pico, Module:RaspberryPi_Pico_SMD, symbol MCU_Module:RaspberryPi_Pico_Extensive
- added Stick_L1: Thumbstick_L, Connector_PinHeader_2.54mm:PinHeader_1x05_P2.54mm_Vertical, symbol Connector_Generic:Conn_01x05
- added Stick_R1: Thumbstick_R, Connector_PinHeader_2.54mm:PinHeader_1x05_P2.54mm_Vertical, symbol Connector_Generic:Conn_01x05
- added Trig_L1: AS5600_L_Trigger, Connector_PinHeader_2.54mm:PinHeader_1x04_P2.54mm_Vertical, symbol Connector_Generic:Conn_01x04
- added Trig_R1: AS5600_R_Trigger, Connector_PinHeader_2.54mm:PinHeader_1x04_P2.54mm_Vertical, symbol Connector_Generic:Conn_01x04
Connections:
- new net +3V3: C1.1, C2.1, C3.1, C4.1, C5.1, C6.1, R1.2, R10.2, R11.2, R12.2, R13.2, R14.2, R15.2, R16.2, R2.2, R3.2, R4.2, R5.2, R6.2, R7.2, R8.2, R9.2, RP1.36 (3V3), Stick_L1.1 (Pin_1), Stick_R1.1 (Pin_1), Trig_L1.1 (Pin_1), Trig_R1.1 (Pin_1)
- new net +5V_USB: C7.1, C8.1, LED1.1 (VDD), LED2.1 (VDD), LED3.1 (VDD), LED4.1 (VDD), LED5.1 (VDD), LED6.1 (VDD), LED7.1 (VDD), LED8.1 (VDD), RP1.39 (VSYS), RP1.40 (VBUS)
- new net ADC0_LSTICK_X: RP1.31 (GPIO26_ADC0), Stick_L1.3 (Pin_3)
- new net ADC1_LSTICK_Y: RP1.32 (GPIO27_ADC1), Stick_L1.2 (Pin_2)
- new net ADC3_RSTICK_X: RP1.14 (GPIO10), Stick_R1.3 (Pin_3)
- new net ADC4_RSTICK_Y: RP1.15 (GPIO11), Stick_R1.2 (Pin_2)
- new net BTN_A: Bt_R_A1.1, Bt_R_A1.2, R5.1, RP1.17 (GPIO13)
- new net BTN_B: Bt_R_B1.1, Bt_R_B1.2, R6.1, RP1.19 (GPIO14)
- new net BTN_GUIDE: Bt_Guide1.1, Bt_Guide1.2, R13.1, RP1.25 (GPIO19)
- new net BTN_LB: Bt_L_LB1.1, Bt_L_LB1.2, R9.1, RP1.11 (GPIO8)
- new net BTN_LS: R15.1, RP1.26 (GPIO20), Stick_L1.4 (Pin_4)
- new net BTN_MENU: Bt_Menu1.1, Bt_Menu1.2, R11.1, RP1.22 (GPIO17)
- new net BTN_RB: Bt_R_RB1.1, Bt_R_RB1.2, R10.1, RP1.12 (GPIO9)
- new net BTN_RS: R16.1, RP1.27 (GPIO21), Stick_R1.4 (Pin_4)
- new net BTN_SHARE: Bt_Share1.1, Bt_Share1.2, R14.1, RP1.16 (GPIO12)
- new net BTN_VIEW: Bt_View1.1, Bt_View1.2, R12.1, RP1.24 (GPIO18)
- new net BTN_X: Bt_R_X1.1, Bt_R_X1.2, R7.1, RP1.20 (GPIO15)
- new net BTN_Y: Bt_R_Y1.1, Bt_R_Y1.2, R8.1, RP1.21 (GPIO16)
- new net DPAD_DOWN: Bt_L_S1.3, Bt_L_S1.4, R2.1, RP1.5 (GPIO3)
- new net DPAD_LEFT: Bt_L_A1.3, Bt_L_A1.4, R3.1, RP1.9 (GPIO6)
- new net DPAD_RIGHT: Bt_L_D1.3, Bt_L_D1.4, R4.1, RP1.10 (GPIO7)
- new net DPAD_UP: Bt_L_W1.3, Bt_L_W1.4, R1.1, RP1.4 (GPIO2)
- new net GND: Bt_Guide1.3, Bt_Guide1.4, Bt_L_A1.1, Bt_L_A1.2, Bt_L_D1.1, Bt_L_D1.2, Bt_L_LB1.3, Bt_L_LB1.4, Bt_L_S1.1, Bt_L_S1.2, Bt_L_W1.1, Bt_L_W1.2, Bt_Menu1.3, Bt_Menu1.4, Bt_R_A1.3, Bt_R_A1.4, Bt_R_B1.3, Bt_R_B1.4, Bt_R_RB1.3, Bt_R_RB1.4, Bt_R_X1.3, Bt_R_X1.4, Bt_R_Y1.3, Bt_R_Y1.4, Bt_Share1.3, Bt_Share1.4, Bt_View1.3, Bt_View1.4, C1.2, C2.2, C3.2, C4.2, C5.2, C6.2, C7.2, C8.2, LED1.3 (VSS), LED2.3 (VSS), LED3.3 (VSS), LED4.3 (VSS), LED5.3 (VSS), LED6.3 (VSS), LED7.3 (VSS), LED8.3 (VSS), RP1.13 (GND), RP1.18 (GND), RP1.23 (GND), RP1.28 (GND), RP1.3 (GND), RP1.33 (AGND), RP1.38 (GND), RP1.8 (GND), RP1.D2 (GND), RP1.TP1 (USB_GND), Stick_L1.5 (Pin_5), Stick_R1.5 (Pin_5), Trig_L1.2 (Pin_2), Trig_R1.2 (Pin_2)
- new net I2C0_SCL: RP1.2 (GPIO1), Trig_L1.4 (Pin_4)
- new net I2C0_SDA: RP1.1 (GPIO0), Trig_L1.3 (Pin_3)
- new net I2C1_SCL: RP1.7 (GPIO5), Trig_R1.4 (Pin_4)
- new net I2C1_SDA: RP1.6 (GPIO4), Trig_R1.3 (Pin_3)
- new net LED1_2: LED1.2 (DOUT), LED2.4 (DIN)
- new net LED2_3: LED2.2 (DOUT), LED3.4 (DIN)
- new net LED3_4: LED3.2 (DOUT), LED4.4 (DIN)
- new net LED4_5: LED4.2 (DOUT), LED5.4 (DIN)
- new net LED5_6: LED5.2 (DOUT), LED6.4 (DIN)
- new net LED6_7: LED6.2 (DOUT), LED7.4 (DIN)
- new net LED7_8: LED7.2 (DOUT), LED8.4 (DIN)
- new net WS2812_DIN: LED1.4 (DIN), R17.2
- new net WS2812_GP22: R17.1, RP1.29 (GPIO22)
- no-connect marks 0 -> 12
Other:
- title: (none) -> Game Controller Main Board
